Commit message: Implemented secure mechanisms to prevent erratical poses

File: src/pkg_description/urdf/arm/franka_arm.ros2_control.xacro (robot description, xacro)
@@ -22,23 +22,23 @@
           <param name="robot_type">${robot_type}</param>
           <param name="prefix">${arm_prefix}</param>
-          <xacro:if value="${use_fake_hardware}">
-            <!-- <plugin>mock_components/GenericSystem</plugin> -->
-            <plugin>gz_ros2_control/GazeboSimSystem</plugin>
-            <param name="fake_sensor_commands">${fake_sensor_commands}</param>
-            <param name="state_following_offset">0.0</param>
-          </xacro:if>
+          <!-- Gazebo simulation -->
           <xacro:if value="${gazebo}">
             <plugin>gz_ros2_control/GazeboSimSystem</plugin>
-            <!-- <plugin>ign_ros2_control/IgnitionSystem</plugin> -->
+            <param name="position_proportional_gain">30.0</param>
           </xacro:if>
+          <!-- Fake hardware fuera de Gazebo -->
           <xacro:unless value="${gazebo}">
-            <plugin>mock_components/GenericSystem</plugin>
-            <param name="fake_sensor_commands">${fake_sensor_commands}</param>
+            <xacro:if value="${use_fake_hardware}">
+              <plugin>mock_components/GenericSystem</plugin>
+              <param name="fake_sensor_commands">${fake_sensor_commands}</param>
+              <param name="state_following_offset">0.0</param>
+            </xacro:if>
+            <!-- Hardware real fuera de Gazebo -->
+            <xacro:unless value="${use_fake_hardware}">
+              <plugin>franka_hardware/FrankaHardwareInterface</plugin>
+              <param name="robot_ip">${robot_ip}</param>
+              <param name="arm_prefix">${arm_prefix}</param>
+            </xacro:unless>
           </xacro:unless>
-          <xacro:if value="${use_fake_hardware == 0 and gazebo == 0}">
-            <plugin>franka_hardware/FrankaHardwareInterface</plugin>
-            <param name="robot_ip">${robot_ip}</param>
-            <param name="arm_prefix">${arm_prefix}</param>
-          </xacro:if>
         </hardware>
       <!-- Joint position, velocity and effort interfaces -->
@@ -71,5 +71,6 @@
       <xacro:configure_joint joint_name="${arm_prefix}${robot_type}_joint7" initial_position="${pi/4}"/>
       <xacro:if value="${gazebo and hand}">
-        <xacro:configure_joint joint_name="${arm_prefix}${robot_type}_finger_joint1" initial_position="0.0" />
+        <xacro:configure_joint joint_name="${arm_prefix}${robot_type}_finger_joint1" initial_position="0.04" />
+        <xacro:configure_joint joint_name="${arm_prefix}${robot_type}_finger_joint2" initial_position="0.04" />
       </xacro:if>
       <xacro:macro name="general_purpose_io" params="prefix command_interface index">

File: src/pkg_description/urdf/end_effectors/franka_hand/franka_hand.xacro (robot description, xacro)
@@ -113,19 +113,31 @@
     </link>
     <joint name="${ee_prefix}finger_joint1" type="prismatic">
-      <parent link="${ee_prefix}hand" />
-      <child link="${ee_prefix}leftfinger" />
-      <origin xyz="0 0 0.0584" rpy="0 0 0" />
-      <axis xyz="0 1 0" />
-      <limit effort="100" lower="0.0" upper="0.04" velocity="0.2" />
-      <dynamics damping="0.3" />
+      <parent link="${ee_prefix}hand"/>
+      <child link="${ee_prefix}leftfinger"/>
+      <origin xyz="0 0 0.0584" rpy="0 0 0"/>
+      <axis xyz="0 1 0"/>
+      <xacro:if value="${gazebo}">
+        <limit effort="100" lower="0.003" upper="0.04" velocity="0.2"/>
+      </xacro:if>
+      <xacro:unless value="${gazebo}">
+        <limit effort="100" lower="0.0" upper="0.04" velocity="0.2"/>
+      </xacro:unless>
+      <dynamics damping="0.01" friction="0.0"/>
     </joint>
     <joint name="${ee_prefix}finger_joint2" type="prismatic">
-      <parent link="${ee_prefix}hand" />
-      <child link="${ee_prefix}rightfinger" />
-      <origin xyz="0 0 0.0584" rpy="0 0 ${pi}" />
-      <axis xyz="0 1 0" />
-      <limit effort="100" lower="0.0" upper="0.04" velocity="0.2" />
-      <mimic joint="${ee_prefix}finger_joint1" />
-      <dynamics damping="0.3" />
+      <parent link="${ee_prefix}hand"/>
+      <child link="${ee_prefix}rightfinger"/>
+      <origin xyz="0 0 0.0584" rpy="0 0 ${pi}"/>
+      <axis xyz="0 1 0"/>
+      <xacro:if value="${gazebo}">
+        <limit effort="100" lower="0.003" upper="0.04" velocity="0.2"/>
+      </xacro:if>
+      <xacro:unless value="${gazebo}">
+        <limit effort="100" lower="0.0" upper="0.04" velocity="0.2"/>
+      </xacro:unless>
+      <xacro:unless value="${gazebo}">
+        <mimic joint="${ee_prefix}finger_joint1"/>
+      </xacro:unless>
+      <dynamics damping="0.01" friction="0.0"/>
     </joint>
   </xacro:macro>
